Commit message: Integrate SolidWorks sentry model and navigation workflow

File: src/sentry_description/urdf/mid360.xacro (robot description, xacro)
@@ -1,6 +1,7 @@
 <?xml version="1.0"?>
 <robot xmlns:xacro="http://www.ros.org/wiki/xacro">
- <xacro:macro name="sentry_mid360" params="mount_x mount_y mount_z mount_pitch">
+ <xacro:macro name="sentry_mid360" params="mount_x mount_y mount_z mount_pitch show_visual:=true">
   <link name="lidar_link">
+   <xacro:if value="${show_visual}">
    <visual>
     <origin rpy="1.570796 0 -1.570796"/>
@@ -8,4 +9,5 @@
     <material name="mid360_orange"><color rgba="1.0 0.20 0.02 1.0"/></material>
    </visual>
+   </xacro:if>
   </link>
   <joint name="lidar_joint" type="fixed"><parent link="gimbal_yaw_link"/><child link="lidar_link"/><origin xyz="${mount_x} ${mount_y} ${mount_z}" rpy="0 ${mount_pitch} 0"/></joint>

File: src/sentry_description/urdf/sentry.urdf.xacro (robot description, xacro)
@@ -2,29 +2,43 @@
 <robot xmlns:xacro="http://www.ros.org/wiki/xacro" name="sentry">
  <xacro:arg name="use_gazebo" default="false"/>
+ <xacro:arg name="use_solidworks" default="true"/>
  <xacro:include filename="$(find sentry_description)/urdf/chassis.xacro"/>
  <xacro:include filename="$(find sentry_description)/urdf/wheels.xacro"/>
  <xacro:include filename="$(find sentry_description)/urdf/gimbal.xacro"/>
+ <xacro:include filename="$(find sentry_description)/urdf/solidworks.xacro"/>
  <xacro:include filename="$(find sentry_description)/urdf/mid360.xacro"/>
  <xacro:include filename="$(find sentry_description)/urdf/gazebo.xacro"/>
- <!-- APPROXIMATE first-pass geometry; calibrate these values in RViz. -->
  <xacro:property name="wheel_radius" value="0.0775"/>
- <xacro:property name="wheel_width" value="0.050"/>
-<!-- Equal X/Y mounting offsets yield a 450 mm wheel-centre diagonal. -->
-<xacro:property name="wheel_x" value="0.1331"/><xacro:property name="wheel_y" value="0.1331"/>
  <link name="base_footprint"/>
  <joint name="base_footprint_joint" type="fixed"><parent link="base_footprint"/><child link="base_link"/>
   <origin xyz="0 0 ${wheel_radius}"/></joint>
- <xacro:sentry_chassis/>
-<!--
-  The wheel STL includes its suspension arm.  From the CAD top view, its four
-  mounting corners use the CAD-specific orientations below.  The left pair is
-  flipped 180 degrees relative to the initial visual calibration.
--->
-<xacro:sentry_wheel prefix="fl" x="${wheel_x}" y="${wheel_y}" yaw="2.356194"/>
-<xacro:sentry_wheel prefix="fr" x="${wheel_x}" y="${-wheel_y}" yaw="0.785398"/>
-<xacro:sentry_wheel prefix="rl" x="${-wheel_x}" y="${wheel_y}" yaw="-2.356194"/>
-<xacro:sentry_wheel prefix="rr" x="${-wheel_x}" y="${-wheel_y}" yaw="-0.785398"/>
- <xacro:sentry_gimbal mount_z="0.177" mount_yaw="1.570796"/>
- <xacro:sentry_mid360 mount_x="-0.145" mount_y="-0.01" mount_z="0.110" mount_pitch="-0.610865"/>
+ <xacro:if value="$(arg use_solidworks)">
+  <xacro:solidworks_chassis/>
+  <xacro:solidworks_armor index="1" x="0.23985" y="0" z="0.063281" yaw="0"/>
+  <xacro:solidworks_armor index="2" x="0" y="0.23985" z="0.097281" yaw="1.5708"/>
+  <xacro:solidworks_armor index="3" x="-0.23985" y="0" z="0.063281" yaw="3.1416"/>
+  <xacro:solidworks_armor index="4" x="0" y="-0.23985" z="0.097281" yaw="-1.5708"/>
+  <!-- SolidWorks wheel numbering is FL, RL, RR, FR. -->
+  <xacro:solidworks_wheel prefix="fl" index="1" x="0.16209" y="0.16209" yaw="0.7854"/>
+  <xacro:solidworks_wheel prefix="fr" index="4" x="0.16209" y="-0.16209" yaw="-0.7854"/>
+  <xacro:solidworks_wheel prefix="rl" index="2" x="-0.16209" y="0.16209" yaw="2.3562"/>
+  <xacro:solidworks_wheel prefix="rr" index="3" x="-0.16209" y="-0.16209" yaw="-2.3562"/>
+  <xacro:solidworks_gimbal/>
+  <!-- The CAD yaw mesh already contains the MID360 exterior. Keep its sensor TF. -->
+  <xacro:sentry_mid360 mount_x="-0.145" mount_y="-0.01" mount_z="0.110"
+                       mount_pitch="-0.610865" show_visual="false"/>
+ </xacro:if>
+ <xacro:unless value="$(arg use_solidworks)">
+  <xacro:property name="wheel_x" value="0.1331"/>
+  <xacro:property name="wheel_y" value="0.1331"/>
+  <xacro:sentry_chassis/>
+  <xacro:sentry_wheel prefix="fl" x="${wheel_x}" y="${wheel_y}" yaw="2.356194"/>
+  <xacro:sentry_wheel prefix="fr" x="${wheel_x}" y="${-wheel_y}" yaw="0.785398"/>
+  <xacro:sentry_wheel prefix="rl" x="${-wheel_x}" y="${wheel_y}" yaw="-2.356194"/>
+  <xacro:sentry_wheel prefix="rr" x="${-wheel_x}" y="${-wheel_y}" yaw="-0.785398"/>
+  <xacro:sentry_gimbal mount_z="0.177" mount_yaw="1.570796"/>
+  <xacro:sentry_mid360 mount_x="-0.145" mount_y="-0.01" mount_z="0.110"
+                       mount_pitch="-0.610865"/>
+ </xacro:unless>
  <xacro:sentry_gazebo enabled="$(arg use_gazebo)"/>
 </robot>
